File: ControlLEDs.kicad_sch (KiCad schematic)
At the start: 16 parts

Commit message: finished schematic rev1
Parts:
- removed D10: M_CNCTR, Diode_SMD:D_0805_2012Metric, symbol Device:LED
- removed D2: BPS_PWR, Diode_SMD:D_0805_2012Metric, symbol Device:LED
- removed D3: LEFT_BLINK, Diode_SMD:D_0805_2012Metric, symbol Device:LED
- removed D4: BPS_FAULT, Diode_SMD:D_0805_2012Metric, symbol Device:LED
- removed D5: A_CNCTR, Diode_SMD:D_0805_2012Metric, symbol Device:LED
- removed D7: RIGHT_BLINK, Diode_SMD:D_0805_2012Metric, symbol Device:LED
- removed R2, R5: 680, Resistor_SMD:R_0805_2012Metric, symbol Device:R
- removed R3, R7: 390, Resistor_SMD:R_0805_2012Metric, symbol Device:R
- removed R4: 5k, Resistor_SMD:R_0805_2012Metric, symbol Device:R
- added D9: RIGHT_BLINK, Diode_SMD:D_0805_2012Metric, symbol Device:LED
- added J4, J5, J6: Conn_01x02, Connector_Molex:Molex_Micro-Fit_3.0_43650-0200_1x02_P3.00mm_Horizontal, symbol Connector_Generic:Conn_01x02
- added Q3, Q4, Q5: BSD235C, Package_TO_SOT_SMD:SOT-363_SC-70-6, symbol Transistor_FET:BSD235C
- D8: value CTRL_FAULT -> LEFT_BLINK
- renumbered D6 to D7, R8 to R11, R6 to R12
Connections:
- net CTRL_FAULT is gone; now on net LEFT_BLINK: R11.1
- net M_CNCTR is gone; now on net RIGHT_BLINK: R10.1
- net GND: now also D9.1 (K)
- net GNDPWR: now also J4.2 (Pin_2), J5.2 (Pin_2), J6.2 (Pin_2)
- net Headlight_ON: now also Q5.2 (GN)
- net LEFT_BLINK: now also Q4.2 (GN)
- net RIGHT_BLINK: now also Q3.2 (GN)
- net at R10.2: now also D9.2 (A)
- new net: J5.1 (Pin_1), Q4.6 (DN)
- new net: J4.1 (Pin_1), Q3.6 (DN)
- new net: J6.1 (Pin_1), Q5.6 (DN)
- new net +12V: Q3.1 (SN), Q4.1 (SN), Q5.1 (SN)
Other:
- note added: "For all resistor values, the assumed output high voltage is 3.3 V and output low voltage is 0.6 V. Standard LED operating point is 1.9 V at 2 mA"
- note removed: "For all resistor values (other than BPS_FAULT), the assumed output high voltage is 3.3 V and output low voltage is 0.6 V. Standard LED operating point is 1.9 V at 2 mA."
- note removed: "Voltage drop from BPS_FAULT+ to BPS_FAULT- is assumed to be 12 V."
- moved on the sheet: D7, D8, R10, R11, R12
