File: PowerDist.kicad_sch (KiCad schematic)
At the start: 8 parts, among them U5 NCP1117-3.3_SOT223

Commit message: finished schematic rev1
Parts:
- renumbered D1 to D0
Changed lines of the file:
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@@
+    (stroke (width 0) (type default) (color 0 0 0 0))
+  )
+  (wire (pts (xy 190.5 97.79) (xy 199.39 97.79))
     (stroke (width 0) (type default) (color 0 0 0 0))
   )
@@
   )
   (wire (pts (xy 138.43 91.44) (xy 129.54 91.44))
-    (stroke (width 0) (type default) (color 0 0 0 0))
-  )
-  (wire (pts (xy 190.5 97.79) (xy 199.39 97.79))
     (stroke (width 0) (type default) (color 0 0 0 0))
   )
@@
     (effects (font (size 1.27 1.27)) (justify left))
   )
-  (hierarchical_label "+3.3V" (shape input) (at 209.55 97.79 0)
+  (hierarchical_label "+3V3" (shape input) (at 209.55 97.79 0)
     (effects (font (size 1.27 1.27)) (justify left))
   )
@@
   (symbol (lib_id "Device:LED") (at 129.54 111.76 90) (unit 1)
     (in_bom yes) (on_board yes)
-    (property "Reference" "D1" (id 0) (at 132.5372 110.7694 90)
+    (property "Reference" "D0" (id 0) (at 132.5372 110.7694 90)
       (effects (font (size 1.27 1.27)) (justify right))
     )
