File: BlinkTimer.kicad_sch (KiCad schematic)
At the start: 5 parts

Commit message: finished schematic rev1
Parts:
- C1: renamed from C1_T?; footprint (none) -> Capacitor_SMD:C_0805_2012Metric
- C2: renamed from C2_T?; footprint (none) -> Capacitor_SMD:C_0805_2012Metric
- R22: renamed from R1_T?; footprint (none) -> Resistor_SMD:R_0805_2012Metric
- R23: renamed from R2_T?; footprint (none) -> Resistor_SMD:R_0805_2012Metric
- gave numbers to parts that had none: 1
Connections:
- net LIGHTSCLK renamed OUTCLK
Changed lines of the file:
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@@
 (kicad_sch (version 20211123) (generator eeschema)
   (paper "A4")
-  (junction (at 170.815 85.09) (diameter 0) (color 0 0 0 0)
-  )
   (junction (at 170.815 101.6) (diameter 0) (color 0 0 0 0)
   )
   (junction (at 170.815 96.52) (diameter 0) (color 0 0 0 0)
   )
-  (junction (at 170.815 113.03) (diameter 0) (color 0 0 0 0)
-  )
-  (wire (pts (xy 170.815 113.03) (xy 173.99 113.03))
-    (stroke (width 0) (type default) (color 0 0 0 0))
-  )
   (wire (pts (xy 129.54 96.52) (xy 130.175 96.52))
     (stroke (width 0) (type default) (color 0 0 0 0))
@@
     (stroke (width 0) (type default) (color 0 0 0 0))
   )
-  (wire (pts (xy 170.815 114.3) (xy 170.815 113.03))
-    (stroke (width 0) (type default) (color 0 0 0 0))
-  )
   (wire (pts (xy 130.175 105.41) (xy 130.175 101.6))
     (stroke (width 0) (type default) (color 0 0 0 0))
@@
     (stroke (width 0) (type default) (color 0 0 0 0))
   )
-  (wire (pts (xy 173.355 85.09) (xy 170.815 85.09))
-    (stroke (width 0) (type default) (color 0 0 0 0))
-  )
   (wire (pts (xy 155.575 101.6) (xy 170.815 101.6))
     (stroke (width 0) (type default) (color 0 0 0 0))
@@
     (stroke (width 0) (type default) (color 0 0 0 0))
   )
-  (wire (pts (xy 170.815 113.03) (xy 170.815 111.125))
+  (wire (pts (xy 170.815 111.125) (xy 170.815 114.3))
     (stroke (width 0) (type default) (color 0 0 0 0))
   )
@@
     (effects (font (size 1.27 1.27)) (justify right bottom))
   )
-  (hierarchical_label "GND" (shape input) (at 173.99 113.03 0)
+  (hierarchical_label "OUTCLK" (shape input) (at 157.48 91.44 0)
     (effects (font (size 1.27 1.27)) (justify left))
   )
-  (hierarchical_label "LIGHTSCLK" (shape input) (at 157.48 91.44 0)
-    (effects (font (size 1.27 1.27)) (justify left))
-  )
-  (hierarchical_label "+3.3v" (shape input) (at 173.355 85.09 0)
-    (effects (font (size 1.27 1.27)) (justify left))
-  )
   (symbol (lib_id "Device:R_Small") (at 170.815 91.44 0) (unit 1)
     (in_bom yes) (on_board yes) (fields_autoplaced)
-    (property "Reference" "R1_T?" (id 0) (at 172.72 90.1699 0)
+    (property "Reference" "R22" (id 0) (at 172.72 90.1699 0)
       (effects (font (size 1.27 1.27)) (justify left))
     )
@@
       (effects (font (size 1.27 1.27)) (justify left))
     )
-    (property "Footprint" "" (id 2) (at 170.815 91.44 0)
+    (property "Footprint" "Resistor_SMD:R_0805_2012Metric" (id 2) (at 170.815 91.44 0)
       (effects (font (size 1.27 1.27)) hide)
     )
@@
   (symbol (lib_id "power:+3.3V") (at 170.815 85.09 0) (unit 1)
     (in_bom yes) (on_board yes) (fields_autoplaced)
-    (property "Reference" "#PWR?" (id 0) (at 170.815 88.9 0)
+    (property "Reference" "#PWR0136" (id 0) (at 170.815 88.9 0)
       (effects (font (size 1.27 1.27)) hide)
     )
@@
   (symbol (lib_id "Device:C_Small") (at 127 96.52 270) (unit 1)
     (in_bom yes) (on_board yes)
-    (property "Reference" "C1_T?" (id 0) (at 127 100.33 90))
+    (property "Reference" "C1" (id 0) (at 127 100.33 90))
     (property "Value" "10uF" (id 1) (at 127 102.87 90))
-    (property "Footprint" "" (id 2) (at 127 96.52 0)
+    (property "Footprint" "Capacitor_SMD:C_0805_2012Metric" (id 2) (at 127 96.52 0)
       (effects (font (size 1.27 1.27)) hide)
     )
@@
   (symbol (lib_id "power:GND") (at 142.875 106.68 0) (unit 1)
     (in_bom yes) (on_board yes) (fields_autoplaced)
-    (property "Reference" "#PWR?" (id 0) (at 142.875 113.03 0)
+    (property "Reference" "#PWR0134" (id 0) (at 142.875 113.03 0)
       (effects (font (size 1.27 1.27)) hide)
     )
@@
   (symbol (lib_id "power:GND") (at 170.815 114.3 0) (unit 1)
     (in_bom yes) (on_board yes) (fields_autoplaced)
-    (property "Reference" "#PWR?" (id 0) (at 170.815 120.65 0)
+    (property "Reference" "#PWR0132" (id 0) (at 170.815 120.65 0)
       (effects (font (size 1.27 1.27)) hide)
     )
@@
   (symbol (lib_id "power:+3.3V") (at 130.175 105.41 180) (unit 1)
     (in_bom yes) (on_board yes) (fields_autoplaced)
-    (property "Reference" "#PWR?" (id 0) (at 130.175 101.6 0)
+    (property "Reference" "#PWR0135" (id 0) (at 130.175 101.6 0)
       (effects (font (size 1.27 1.27)) hide)
     )
@@
   (symbol (lib_id "Device:R_Small") (at 170.815 99.06 180) (unit 1)
     (in_bom yes) (on_board yes) (fields_autoplaced)
-    (property "Reference" "R2_T?" (id 0) (at 172.72 97.7899 0)
+    (property "Reference" "R23" (id 0) (at 172.72 97.7899 0)
       (effects (font (size 1.27 1.27)) (justify right))
     )
@@
       (effects (font (size 1.27 1.27)) (justify right))
     )
-    (property "Footprint" "" (id 2) (at 170.815 99.06 0)
+    (property "Footprint" "Resistor_SMD:R_0805_2012Metric" (id 2) (at 170.815 99.06 0)
       (effects (font (size 1.27 1.27)) hide)
     )
@@
   (symbol (lib_id "power:+3.3V") (at 142.875 86.36 0) (unit 1)
     (in_bom yes) (on_board yes) (fields_autoplaced)
-    (property "Reference" "#PWR?" (id 0) (at 142.875 90.17 0)
+    (property "Reference" "#PWR0133" (id 0) (at 142.875 90.17 0)
       (effects (font (size 1.27 1.27)) hide)
     )
@@
   (symbol (lib_id "power:GND") (at 124.46 96.52 270) (unit 1)
     (in_bom yes) (on_board yes) (fields_autoplaced)
-    (property "Reference" "#PWR?" (id 0) (at 118.11 96.52 0)
+    (property "Reference" "#PWR0137" (id 0) (at 118.11 96.52 0)
       (effects (font (size 1.27 1.27)) hide)
     )
@@
   (symbol (lib_id "Device:C_Small") (at 170.815 108.585 0) (unit 1)
     (in_bom yes) (on_board yes) (fields_autoplaced)
-    (property "Reference" "C2_T?" (id 0) (at 173.99 107.3212 0)
+    (property "Reference" "C2" (id 0) (at 173.99 107.3212 0)
       (effects (font (size 1.27 1.27)) (justify left))
     )
@@
       (effects (font (size 1.27 1.27)) (justify left))
     )
-    (property "Footprint" "" (id 2) (at 170.815 108.585 0)
+    (property "Footprint" "Capacitor_SMD:C_0805_2012Metric" (id 2) (at 170.815 108.585 0)
       (effects (font (size 1.27 1.27)) hide)
     )
@@
   (symbol (lib_id "Timer:LM555xM") (at 142.875 96.52 0) (unit 1)
     (in_bom yes) (on_board yes) (fields_autoplaced)
-    (property "Reference" "BlinkTimer?" (id 0) (at 144.8944 83.82 0)
-      (effects (font (size 1.27 1.27)) (justify left))
-    )
+    (property "Reference" "BL1" (id 0) (at 144.8944 83.82 0)
+      (effects (font (size 1.27 1.27)) (justify left))
+    )

Commit message: redo schematic
Parts:
- added U?: NCP1117-3.3_SOT223, Package_TO_SOT_SMD:SOT-223-3_TabPin2, symbol Regulator_Linear:NCP1117-3.3_SOT223
Connections:
- net GND: now also U?.1 (GND); no longer BL1.1 (GND), C1.2, C2.2
- net OUTCLK: now also U?.2 (VO); no longer BL1.3 (Q)
- net +3V3 renamed +12V
- net +12V: no longer BL1.4 (R)
- new net +5V: BL1.4 (R)
- new net GNDPWR: BL1.1 (GND), C1.2, C2.2
- new net OUTCLK_5: BL1.3 (Q), U?.3 (VI)

Commit message: added todo
Parts:
- removed U?: NCP1117-3.3_SOT223, Package_TO_SOT_SMD:SOT-223-3_TabPin2, symbol Regulator_Linear:NCP1117-3.3_SOT223
Connections:
- net +5V is gone; now on net +12V: BL1.4 (R)
- net OUTCLK_5 is gone; now on net OUTCLK: BL1.3 (Q)
Changed lines of the file:
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@@
-    (stroke (width 0) (type default) (color 0 0 0 0))
-  )
-  (wire (pts (xy 193.04 109.22) (xy 193.04 104.775))
     (stroke (width 0) (type default) (color 0 0 0 0))
   )
@@
     (effects (font (size 1.27 1.27)) (justify left bottom))
   )
-  (label "OUTCLK_5" (at 157.48 91.44 0)
-    (effects (font (size 1.27 1.27)) (justify left bottom))
-  )
-  (label "OUTCLK_5" (at 193.04 109.22 0)
-    (effects (font (size 1.27 1.27)) (justify left bottom))
-  )
   (label "TRIGTHRES" (at 155.575 101.6 0)
     (effects (font (size 1.27 1.27)) (justify left bottom))
@@
     (effects (font (size 1.27 1.27)) (justify right bottom))
   )
-  (hierarchical_label "OUTCLK" (shape input) (at 193.04 89.535 90)
+  (hierarchical_label "OUTCLK" (shape input) (at 157.48 91.44 0)
     (effects (font (size 1.27 1.27)) (justify left))
   )
@@
     (pin "2")
   )
-  (symbol (lib_id "power:GND") (at 200.66 97.155 90) (unit 1)
-    (in_bom yes) (on_board yes) (fields_autoplaced)
-    (property "Reference" "#PWR?" (id 0) (at 207.01 97.155 0)
-      (effects (font (size 1.27 1.27)) hide)
-    )
-    (property "Value" "GND" (id 1) (at 204.47 97.1549 90)
-      (effects (font (size 1.27 1.27)) (justify right))
-    )
-    (property "Footprint" "" (id 2) (at 200.66 97.155 0)
-      (effects (font (size 1.27 1.27)) hide)
-    )
-    (property "Datasheet" "" (id 3) (at 200.66 97.155 0)
-      (effects (font (size 1.27 1.27)) hide)
-    )
-    (pin "1")
-  )
-  (symbol (lib_id "power:+5V") (at 130.175 105.41 180) (unit 1)
-    (in_bom yes) (on_board yes) (fields_autoplaced)
-    (property "Reference" "#PWR0133" (id 0) (at 130.175 101.6 0)
-      (effects (font (size 1.27 1.27)) hide)
-    )
-    (property "Value" "+5V" (id 1) (at 130.175 110.49 0))
-    (property "Footprint" "" (id 2) (at 130.175 105.41 0)
-      (effects (font (size 1.27 1.27)) hide)
-    )
-    (property "Datasheet" "" (id 3) (at 130.175 105.41 0)
-      (effects (font (size 1.27 1.27)) hide)
-    )
-    (pin "1")
-  )
   (symbol (lib_id "Timer:LM555xM") (at 142.875 96.52 0) (unit 1)
     (in_bom yes) (on_board yes) (fields_autoplaced)
@@
     (pin "6")
     (pin "7")
-  )
-  (symbol (lib_id "Regulator_Linear:NCP1117-3.3_SOT223") (at 193.04 97.155 90) (unit 1)
-    (in_bom yes) (on_board yes)
-    (property "Reference" "U?" (id 0) (at 220.98 99.06 90)
-      (effects (font (size 1.27 1.27)) (justify left))
-    )
-    (property "Value" "NCP1117-3.3_SOT223" (id 1) (at 220.98 101.6 90)
-      (effects (font (size 1.27 1.27)) (justify left))
-    )
-    (property "Footprint" "Package_TO_SOT_SMD:SOT-223-3_TabPin2" (id 2) (at 187.96 97.155 0)
-      (effects (font (size 1.27 1.27)) hide)
-    )
-    (property "Datasheet" "http://www.onsemi.com/pub_link/Collateral/NCP1117-D.PDF" (id 3) (at 199.39 94.615 0)
-      (effects (font (size 1.27 1.27)) hide)
-    )
-    (pin "1")
-    (pin "2")
-    (pin "3")
   )
   (symbol (lib_id "power:+12V") (at 142.875 75.565 0) (unit 1)
@@
       (effects (font (size 1.27 1.27)) hide)
     )
+    (pin "1")
+  )
+  (symbol (lib_id "power:+12V") (at 130.175 105.41 180) (unit 1)
+    (in_bom yes) (on_board yes) (fields_autoplaced)
+    (property "Reference" "#PWR?" (id 0) (at 130.175 101.6 0)
+      (effects (font (size 1.27 1.27)) hide)
+    )
+    (property "Value" "+12V" (id 1) (at 130.175 110.49 0))
+    (property "Footprint" "" (id 2) (at 130.175 105.41 0)
+      (effects (font (size 1.27 1.27)) hide)
+    )
+    (property "Datasheet" "" (id 3) (at 130.175 105.41 0)
+      (effects (font (size 1.27 1.27)) hide)
+    )
