File: Controls-LightingPCB.kicad_pcb (KiCad board)
At the start: 2 copper layers, 63.5 x 114.3 mm, 50 parts, among them J3 MinionConn, SW1 HAZARD, SW2 CRUISE_SET, SW3 CRUISE, SW4 F/R_SW, SW5 HEADLIGHT_SW, SW7 TURN_SIGNAL_SW, SW8 REGEN_SW, U3 MCP23S17_SS, U5 NCP1117-3.3_SOT223

Commit message: finished schematic rev1
Parts:
- removed D10: M_CNCTR, Diode_SMD:D_0805_2012Metric
- removed D5: A_CNCTR, Diode_SMD:D_0805_2012Metric
- removed D6: Headlight_ON, Diode_SMD:D_0805_2012Metric
- removed J3: MinionConn, Connector_Molex:Molex_Micro-Fit_3.0_43650-0900_1x09_P3.00mm_Horizontal
- removed LOGO1: Dr. Hallock Logo, UTSVT_Special:Hallock_Image_Small
- removed LOGO2: UTSVT Logo, UTSVT_Special:UTSVT_Logo_Symbol
- removed R3, R7: 390, Resistor_SMD:R_0805_2012Metric
- removed R4: 5k, Resistor_SMD:R_0805_2012Metric
- removed R5, R6, R8: 680, Resistor_SMD:R_0805_2012Metric
- removed U3: MCP23S17_SS, Package_SO:SSOP-28_5.3x10.2mm_P0.65mm
- added BL1: LM555xM, Package_SO:SOIC-8_3.9x4.9mm_P1.27mm, F.Cu at (93.8, 114.1)
- added C1: 10uF, Capacitor_SMD:C_0805_2012Metric, F.Cu at (91.8, 118.9)
- added C2: 10uF, Capacitor_SMD:C_0805_2012Metric, F.Cu at (104.0, 112.4)
- added D0: PowerOn, LED_SMD:LED_0805_2012Metric, F.Cu at (98.5, 68.0)
- added D9: RIGHT_BLINK, Diode_SMD:D_0805_2012Metric, F.Cu at (89.0, 49.3)
- added J1: MinionConn, Connector_Molex:Molex_Micro-Fit_3.0_43650-0900_1x09_P3.00mm_Horizontal, F.Cu at (74.8, 154.8)
- added J2: Conn_01x02, Connector_Molex:Molex_Micro-Fit_3.0_43650-0200_1x02_P3.00mm_Horizontal, F.Cu at (33.5, 88.4)
- added J4: Conn_01x02, Connector_Molex:Molex_Micro-Fit_3.0_43650-0200_1x02_P3.00mm_Horizontal, F.Cu at (102.8, 42.7)
- added J5: Conn_01x02, Connector_Molex:Molex_Micro-Fit_3.0_43650-0200_1x02_P3.00mm_Horizontal, F.Cu at (91.1, 42.7)
- added J6: Conn_01x02, Connector_Molex:Molex_Micro-Fit_3.0_43650-0200_1x02_P3.00mm_Horizontal, F.Cu at (114.5, 42.7)
- added Q1: BSD235C, Package_TO_SOT_SMD:SOT-363_SC-70-6, F.Cu at (64.0, 75.5)
- added Q2: BSD235C, Package_TO_SOT_SMD:SOT-363_SC-70-6, F.Cu at (74.7, 71.4)
- added Q3: BSD235C, Package_TO_SOT_SMD:SOT-363_SC-70-6, F.Cu at (102.2, 49.6)
- added Q4: BSD235C, Package_TO_SOT_SMD:SOT-363_SC-70-6, F.Cu at (106.4, 46.6)
- added Q5: BSD235C, Package_TO_SOT_SMD:SOT-363_SC-70-6, F.Cu at (110.7, 46.6)
- added R11: 680, Resistor_SMD:R_0805_2012Metric, F.Cu at (97.9, 46.2)
- added R12: 680, Resistor_SMD:R_0805_2012Metric, F.Cu at (93.5, 49.2)
- added R22: 8.2k, Resistor_SMD:R_0805_2012Metric, F.Cu at (100.2, 118.0)
- D1: value PowerOn -> 1N914; footprint LED_SMD:LED_0805_2012Metric -> Diode_THT:D_DO-35_SOD27_P7.62mm_Horizontal; moved to F.Cu
- D2: value BPS_PWR -> 1N914; footprint Diode_SMD:D_0805_2012Metric -> Diode_THT:D_DO-35_SOD27_P7.62mm_Horizontal; moved to F.Cu
- D3: value LEFT_BLINK -> 1N914; footprint Diode_SMD:D_0805_2012Metric -> Diode_THT:D_DO-35_SOD27_P7.62mm_Horizontal; moved to F.Cu
- D4: value BPS_FAULT -> 1N914; footprint Diode_SMD:D_0805_2012Metric -> Diode_THT:D_DO-35_SOD27_P7.62mm_Horizontal; moved to F.Cu
- D7: value RIGHT_BLINK -> Headlight_ON; moved to F.Cu
- D8: value CTRL_FAULT -> LEFT_BLINK; moved to F.Cu
- R1: value 60 -> 10k
- R2: value 680 -> 10k
- R23: value 10k -> 68k
- moved R13 173.9 mm to (31.4, 61.1), turned to 0 degrees
- moved R14 169.5 mm to (31.4, 58.1), turned to 0 degrees
- moved R15 168.5 mm to (35.8, 58.1), turned to 0 degrees
- moved SW2 156.5 mm to (48.2, 42.7), turned to 0 degrees
- moved H4 149.9 mm to (55.4, 82.2)
- moved SW7 147.4 mm to (33.5, 42.7), turned to 0 degrees
- moved R16 146.8 mm to (35.8, 61.1), turned to 0 degrees
- moved D4 143.8 mm to (30.7, 92.2), turned to 0 degrees
- moved H3 143.7 mm to (44.6, 85.8)
- moved SW3 143.7 mm to (48.2, 54.6), turned to 0 degrees
- moved R21 141.3 mm to (44.6, 61.1), turned to 0 degrees
- moved R17 139.2 mm to (40.2, 58.1), turned to 0 degrees
- moved SW1 132.4 mm to (59.9, 42.7), turned to 0 degrees
- moved D2 126.1 mm to (42.4, 80.2)
- moved D1 120.1 mm to (63.4, 71.8)
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Connections:
- D1 pad 1: GND -> Net-(D1-Pad1)
- D1 pad 2: Net-(D1-Pad2) -> /LEFT_SW
- D2 pad 1: GNDPWR -> Net-(D1-Pad1)
- D2 pad 2: Net-(D2-Pad2) -> /HZD_SW
- D3 pad 1: /LEFT_BLINK -> Net-(D3-Pad1)
- D3 pad 2: Net-(D3-Pad2) -> /RIGHT_SW
- D4 pad 1: GNDPWR -> Net-(D3-Pad1)
- D4 pad 2: Net-(D4-Pad2) -> /HZD_SW
- D7 pad 1: /RIGHT_BLINK -> GND
- R1 pad 1: /MISO -> Net-(D1-Pad1)
- R1 pad 2: Net-(J3-Pad4) -> GND
- R10 pad 1: /M_CNCTR -> /RIGHT_BLINK
- R16 pad 1: +3V3 -> GND
- R17 pad 1: +3V3 -> GND
- R18 pad 2: Net-(D1-Pad2) -> Net-(D0-Pad2)
- R19 pad 1: +3V3 -> GND
- R2 pad 1: /BPS_PWR -> Net-(D3-Pad1)
- R2 pad 2: Net-(D2-Pad2) -> GND
- R20 pad 1: +3V3 -> GND
- R23 pad 1: +3V3 -> /BlinkTimer/TRIGTHRES
- SW4 pad 2: GND -> +3V3
- SW7 pad 2: GND -> +3V3
Routing:
- net +3V3: track 266.4 -> 0.00 mm, vias 6 -> 0
- net GNDPWR: track 86.5 -> 0.00 mm, vias 2 -> 0
- net /HZD_SW: track 71.7 -> 0.00 mm, vias 2 -> 0
- net /REV_SW: track 70.6 -> 0.00 mm, vias 4 -> 0
- net /FOR_SW: track 63.1 -> 0.00 mm, vias 2 -> 0
- net /LEFT_BLINK: track 56.9 -> 0.00 mm, vias 1 -> 0
- net /RIGHT_BLINK: track 56.8 -> 0.00 mm, vias 1 -> 0
- net /REGEN_SW: track 54.6 -> 0.00 mm
- net /Headlight_SW: track 53.1 -> 0.00 mm
- net /CRUZ_EN: track 49.9 -> 0.00 mm, vias 1 -> 0
- net /LEFT_SW: track 47.9 -> 0.00 mm
- net /RIGHT_SW: track 46.2 -> 0.00 mm
- net Net-(D2-Pad2): track 46.0 -> 0.00 mm, vias 3 -> 0
- net /CS: track 43.7 -> 0.00 mm
- net /SCK: track 43.0 -> 0.00 mm
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- removed copper zone on B.Cu, net GND
- removed copper zone on F.Cu, net GND
Other:
- board outline removed
- board text removed: "+"
- board text removed: "+3.3 V"
- board text removed: "+5V"
- board text removed: "-"
- board text removed: "Aaron was here"
- board text removed: "Array"
- board text removed: "BPS Fault"
- board text removed: "BPS Power"
- board text removed: "BPS_FAULT+"
- board text removed: "BPS_PWR"
- board text removed: "CLK"
- board text removed: "CS"
- board text removed: "CTRL Fault"
- board text removed: "Cruise Enable"
- board text removed: "Cruise Set"
- board text removed: "Dr. Gary Hallock"
- board text removed: "F/R"
- board text removed: "FOR"
- board text removed: "GND"
- board text removed: "GNDPWR"
- board text removed: "Hazards"
- board text removed: "Head Lights"
- board text removed: "Isha was here"
- board text removed: "Lauren was here"
- board text removed: "Left"
- board text removed: "Left Blink"
- board text removed: "M3"
- board text removed: "MISO"
- board text removed: "MOSI"
- board text removed: "Max was here"
- board text removed: "Minion Conn"
- board text removed: "Motor"
- board text removed: "Power"
- board text removed: "Regen"
- board text removed: "Renee was here"
- board text removed: "Rev"
- board text removed: "Right"
- board text removed: "Right Blink"
- board text removed: "Turn Signal"
- board text removed: "UTSVT - Controls Minion Board v1.4 Fall 2021"
- board text removed: "hi~ :) -nathan"

Commit message: redo schematic
Parts:
- moved R20 227.5 mm to (271.0, 151.6)
- moved H1 196.6 mm to (248.8, 86.2)
- moved H3 191.7 mm to (236.1, 76.0)
- moved H2 185.9 mm to (248.8, 76.0)
- moved H4 180.7 mm to (236.1, 86.2)
- moved R2 160.4 mm to (192.8, 146.9)
- moved D4 160.4 mm to (181.4, 147.2)
- moved D1 136.9 mm to (192.0, 118.9)
- moved D2 136.9 mm to (171.0, 127.3)
- moved D3 136.9 mm to (192.0, 115.4)
- moved Q1 136.9 mm to (192.5, 122.6)
- moved Q2 136.9 mm to (203.3, 118.5)
- moved R1 136.9 mm to (203.4, 115.1)
- moved R13 136.9 mm to (159.9, 108.2)
- moved R14 136.9 mm to (159.9, 105.2)
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
Commit message: PCB layout #1
Parts:
- removed D0: PowerOn, LED_SMD:LED_0805_2012Metric
- removed D9: RIGHT_BLINK, Diode_SMD:D_0805_2012Metric
- removed SW7: TURN_SIGNAL_SW, Connector_Molex:Molex_Micro-Fit_3.0_43650-0300_1x03_P3.00mm_Horizontal
- removed SW8: REGEN_SW, Connector_Molex:Molex_Micro-Fit_3.0_43650-0200_1x02_P3.00mm_Horizontal
- removed U5: NCP1117-3.3_SOT223, Package_TO_SOT_SMD:SOT-223-3_TabPin2
- added C10: .01uF, Capacitor_SMD:C_0805_2012Metric, B.Cu at (261.7, 150.5)
- added C11: .01uF, Capacitor_SMD:C_0805_2012Metric, B.Cu at (251.6, 121.7)
- added C12: C_Small, Capacitor_SMD:C_0805_2012Metric, B.Cu at (258.4, 90.8)
- added C3: .01uF, Capacitor_SMD:C_0805_2012Metric, B.Cu at (251.4, 75.9)
- added C6: 10uF, Capacitor_SMD:C_0805_2012Metric, B.Cu at (258.6, 59.7)
- added C7: .01uF, Capacitor_SMD:C_0805_2012Metric, B.Cu at (251.5, 110.0)
- added C8: .01uF, Capacitor_SMD:C_0805_2012Metric, B.Cu at (260.9, 126.5)
- added C9: 10uF, Capacitor_SMD:C_0805_2012Metric, B.Cu at (253.5, 59.9)
- added D5: SD05_SOD323, Diode_SMD:D_SOD-323, B.Cu at (263.9, 141.0)
- added D6: D_Zener, Diode_SMD:D_0805_2012Metric, B.Cu at (253.5, 51.1)
- added FB1: 12VFB, Inductor_SMD:L_0805_2012Metric, B.Cu at (274.9, 63.2)
- added FB2: GPWRFB, Inductor_SMD:L_0805_2012Metric, B.Cu at (266.4, 41.4)
- added FB3: 5VFB, Inductor_SMD:L_0805_2012Metric, B.Cu at (260.9, 124.2)
- added FB4: GNDFB, Inductor_SMD:L_0805_2012Metric, B.Cu at (244.9, 146.6)
- added FB5: GRBRIDGEFB, Inductor_SMD:L_0805_2012Metric, B.Cu at (263.9, 37.3)
- added HZD_SW1: SPST, Connector_Molex:Molex_Micro-Fit_3.0_43650-0200_1x02_P3.00mm_Horizontal, F.Cu at (247.3, 60.8)
- added J10: INTERNAL_RIGHTBLINK, Connector_Molex:Molex_Micro-Fit_3.0_43650-0200_1x02_P3.00mm_Horizontal, F.Cu at (274.0, 66.4)
- added J11: INTERNAL_LEFTBLINK, Connector_Molex:Molex_Micro-Fit_3.0_43650-0200_1x02_P3.00mm_Horizontal, F.Cu at (274.0, 77.6)
- added J12: EXTERNAL_RIGHTBLINK, Connector_Molex:Molex_Micro-Fit_3.0_43650-0200_1x02_P3.00mm_Horizontal, F.Cu at (274.0, 44.0)
- added J13: EXTERNAL_HDLT, Connector_Molex:Molex_Micro-Fit_3.0_43650-0200_1x02_P3.00mm_Horizontal, F.Cu at (274.0, 100.2)
- added J14: EXTERNAL_BRAKELIGHT, Connector_Molex:Molex_Micro-Fit_3.0_43650-0200_1x02_P3.00mm_Horizontal, F.Cu at (274.0, 88.7)
- added J3: CRUZ_ST_INDICATOR_33v, Connector_Molex:Molex_Micro-Fit_3.0_43650-0200_1x02_P3.00mm_Horizontal, F.Cu at (273.8, 111.9)
- added J7: FOR_INDICATOR_33v, Connector_Molex:Molex_Micro-Fit_3.0_43650-0200_1x02_P3.00mm_Horizontal, F.Cu at (247.3, 128.9)
- added J8: REV_INDICATOR_33v, Connector_Molex:Molex_Micro-Fit_3.0_43650-0200_1x02_P3.00mm_Horizontal, F.Cu at (247.3, 117.4)
- added J9: EXTERNAL_LEFTBLINK, Connector_Molex:Molex_Micro-Fit_3.0_43650-0200_1x02_P3.00mm_Horizontal, F.Cu at (274.0, 55.2)
- added LOGO1: Dr. Hallock Logo, UTSVT_Special:Hallock_Image_Small, F.Cu at (260.0, 122.9)
- added LOGO2: UTSVT Logo, UTSVT_Special:UTSVT_Logo_Symbol, F.Cu at (256.8, 83.1)
- added R24: 0 Ohm, Resistor_SMD:R_0805_2012Metric, B.Cu at (274.9, 73.5)
- added R25: 0 Ohm, Resistor_SMD:R_0805_2012Metric, B.Cu at (274.9, 41.2)
- added R3: 10k, Resistor_SMD:R_0805_2012Metric, B.Cu at (246.5, 87.1)
- added R4: 0k, Resistor_SMD:R_0805_2012Metric, B.Cu at (260.8, 118.9)
- added R5: 0k, Resistor_SMD:R_0805_2012Metric, B.Cu at (260.9, 121.7)
- added R6: 10k, Resistor_SMD:R_0805_2012Metric, B.Cu at (261.0, 129.3)
- added R7: 10k, Resistor_SMD:R_0805_2012Metric, B.Cu at (247.2, 110.0)
- added R8: 6.8k, Resistor_SMD:R_0805_2012Metric, B.Cu at (262.5, 59.7)
- added TP1: GNDPWR_TP, TestPoint:TestPoint_Pad_1.5x1.5mm, F.Cu at (268.5, 103.6)
- added TP2: GND_TP, TestPoint:TestPoint_Pad_1.5x1.5mm, F.Cu at (256.0, 103.6)
- added TP6: 5V_TP, TestPoint:TestPoint_Pad_1.5x1.5mm, F.Cu at (262.1, 103.6)
- added TP7: RIGHT_BLINK_TP, TestPoint:TestPoint_Pad_1.5x1.5mm, F.Cu at (263.7, 107.2)
- added TP8: HDLT_SW, TestPoint:TestPoint_Pad_1.5x1.5mm, F.Cu at (266.7, 107.2)
- added TP9: LIGHTSCLK_TP, TestPoint:TestPoint_Pad_1.5x1.5mm, F.Cu at (257.6, 107.2)
- added U1: NCP1117-3.3_SOT223, Package_TO_SOT_SMD:SOT-223-3_TabPin2, B.Cu at (258.3, 96.3)
- BL1, R2: moved to B.Cu
- C1, C2: value 10uF -> 10u; moved to B.Cu
- C4: value 10u -> .01uF; moved to B.Cu
- C5: value 10u -> 10uF; moved to B.Cu
- D1: value 1N914 -> PowerOn; footprint Diode_THT:D_DO-35_SOD27_P7.62mm_Horizontal -> LED_SMD:LED_0805_2012Metric
- D2, D4: value 1N914 -> 1N5400; footprint Diode_THT:D_DO-35_SOD27_P7.62mm_Horizontal -> Diode_THT:D_DO-201AD_P15.24mm_Horizontal
- D3: value 1N914 -> SD12_SOD323; footprint Diode_THT:D_DO-35_SOD27_P7.62mm_Horizontal -> Diode_SMD:D_SOD-323; moved to B.Cu
- D7: value Headlight_ON -> BAV16W; footprint Diode_SMD:D_0805_2012Metric -> Diode_SMD:D_SOD-123; moved to B.Cu
- D8: value LEFT_BLINK -> BAV16W; footprint Diode_SMD:D_0805_2012Metric -> Diode_SMD:D_SOD-123; moved to B.Cu
- J2: value Conn_01x02 -> 12VPWRCONN
- J4: value Conn_01x02 -> CRUZ_EN_INDICATOR_33v
- J5: value Conn_01x02 -> REGEN_INDICATOR_33v
- J6: value Conn_01x02 -> NEU_INDICATOR_33v
- Q1, Q2, Q3, Q4, Q5: value BSD235C -> 2N7000; footprint Package_TO_SOT_SMD:SOT-363_SC-70-6 -> Package_TO_SOT_THT:TO-92_Inline
- R1: value 10k -> 1.5k; moved to B.Cu
- R10: value 680 -> 0k; moved to B.Cu
- R11, R12: value 680 -> 10k; moved to B.Cu
- R13, R14, R15, R20, R21: value 10k -> 0k; moved to B.Cu
- R16, R17, R19: value 10k -> 100k; moved to B.Cu
- R18: value 1.5k -> 100k; moved to B.Cu
- R22: value 8.2k -> 0 Ohm; moved to B.Cu
- R23: value 68k -> 0 Ohm; moved to B.Cu
- R9: value 10k -> 56k; moved to B.Cu
- SW1: value HAZARD -> CRUISE_SET
- SW2: value CRUISE_SET -> CRUISE_ENABLE
- SW3: value CRUISE -> F/R_SW; footprint Connector_Molex:Molex_Micro-Fit_3.0_43650-0200_1x02_P3.00mm_Horizontal -> Connector_Molex:Molex_Micro-Fit_3.0_43650-0300_1x03_P3.00mm_Horizontal
- SW4: value F/R_SW -> REGEN_SW; footprint Connector_Molex:Molex_Micro-Fit_3.0_43650-0300_1x03_P3.00mm_Horizontal -> Connector_Molex:Molex_Micro-Fit_3.0_43650-0200_1x02_P3.00mm_Horizontal
- SW5: value HEADLIGHT_SW -> TURN_SIGNAL_SW; footprint Connector_Molex:Molex_Micro-Fit_3.0_43650-0200_1x02_P3.00mm_Horizontal -> Connector_Molex:Molex_Micro-Fit_3.0_43650-0300_1x03_P3.00mm_Horizontal
- TP3: value +5V_TP -> 3V3_TP
- TP4: value GND_TP -> LEFT_BLINK_TP
- TP5: value +3.3V_TP -> 12V_TP
- moved SW3 206.3 mm to (273.9, 134.5), turned to -90 degrees
- moved R11 192.2 mm to (259.3, 150.5), turned to 90 degrees
- moved SW4 187.1 mm to (247.3, 72.0)
- moved R22 186.7 mm to (274.9, 51.1), turned to 0 degrees
- moved SW1 182.1 mm to (247.3, 83.2)
- moved R23 178.9 mm to (274.8, 61.2), turned to 0 degrees
- moved SW2 178.4 mm to (247.3, 94.4)
- moved SW5 177.6 mm to (247.3, 49.8)
- moved R18 176.7 mm to (270.6, 67.7), turned to -90 degrees
- moved R12 175.4 mm to (251.6, 125.2), turned to 180 degrees
- moved BL1 174.1 mm to (258.6, 55.6)
- moved D8 172.7 mm to (258.6, 79.0), turned to 180 degrees
- moved TP5 170.2 mm to (265.2, 103.6)
- moved J1 168.2 mm to (272.6, 146.7)
- moved D7 166.6 mm to (258.6, 68.3), turned to 180 degrees
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Connections:
- BL1 pad 2: /BlinkTimer/TRIGTHRES -> /TRIGTHRES
- BL1 pad 4: +3V3 -> +5V
- BL1 pad 6: /BlinkTimer/TRIGTHRES -> /TRIGTHRES
- BL1 pad 8: +3V3 -> +5V
- C1 pad 1: Net-(BL1-Pad5) -> +5V
- C2 pad 1: /BlinkTimer/TRIGTHRES -> +3V3
- C4 pad 1: +5V -> /CRUZ_EN
- C5 pad 1: +3V3 -> Net-(BL1-Pad5)
- D1 pad 1: Net-(D1-Pad1) -> GND
- D1 pad 2: /LEFT_SW -> Net-(D1-Pad2)
- D2 pad 1: Net-(D1-Pad1) -> Net-(D2-Pad1)
- D2 pad 2: /HZD_SW -> Net-(D2-Pad2)
- D3 pad 2: /RIGHT_SW -> Net-(D2-Pad1)
- D4 pad 1: Net-(D3-Pad1) -> Net-(D4-Pad1)
- D4 pad 2: /HZD_SW -> Net-(D4-Pad2)
- D7 pad 1: GND -> /RIGHT_BLINK
- D7 pad 2: Net-(R12-Pad2) -> Net-(D8-Pad2)
- D8 pad 1: GND -> /LEFT_BLINK
- D8 pad 2: Net-(R11-Pad2) -> Net-(D8-Pad2)
- J1 pad 1: +5V -> /EXTRA_CONN
- J1 pad 2: GND -> /BRAKELIGHT
- J1 pad 3: /CRUZ_ST -> /REGEN_SW
- J1 pad 4: /CRUZ_EN -> /FOR_SW
- J1 pad 6: /FOR_SW -> /CRUZ_EN
- J1 pad 7: /REGEN_SW -> /CRUZ_ST
- J1 pad 8: /CONN8 -> Net-(D4-Pad2)
- J1 pad 9: /CONN9 -> Net-(D5-Pad1)
- J2 pad 1: +12V -> Net-(D2-Pad2)
- J2 pad 2: GNDPWR -> Net-(D3-Pad1)
- J4 pad 1: Net-(Q3-Pad6) -> /CRUZ_EN
- J4 pad 2: GNDPWR -> Net-(J4-Pad2)
- J5 pad 1: Net-(Q4-Pad6) -> /REGEN_SW
- J5 pad 2: GNDPWR -> Net-(J5-Pad2)
- J6 pad 1: Net-(Q5-Pad6) -> GND
- J6 pad 2: GNDPWR -> Net-(J6-Pad2)
- Q1 pad 1: /LIGHTSCLK -> GNDPWR
- Q1 pad 2: Net-(D1-Pad1) -> /LEFT_BLINK
- Q1 pad 3: (no net) -> Net-(J9-Pad2)
- Q2 pad 1: /LIGHTSCLK -> GNDPWR
- Q2 pad 2: Net-(D3-Pad1) -> /RIGHT_BLINK
- Q2 pad 3: (no net) -> Net-(J10-Pad2)
- Q3 pad 1: +12V -> GNDPWR
- Q3 pad 2: /RIGHT_BLINK -> /LEFT_BLINK
- Q3 pad 3: (no net) -> Net-(J11-Pad2)
- Q4 pad 1: +12V -> GNDPWR
- Q4 pad 2: /LEFT_BLINK -> /BRAKELIGHT
- Q4 pad 3: (no net) -> Net-(J14-Pad2)
- Q5 pad 1: +12V -> GNDPWR
- Q5 pad 2: /Headlight_SW -> /RIGHT_BLINK
- Q5 pad 3: (no net) -> Net-(J12-Pad2)
- R1 pad 1: Net-(D1-Pad1) -> +5V
- R1 pad 2: GND -> Net-(D1-Pad2)
- R10 pad 1: /RIGHT_BLINK -> Net-(J5-Pad2)
- R10 pad 2: Net-(R10-Pad2) -> GND
- R11 pad 1: /LEFT_BLINK -> GND
- R11 pad 2: Net-(R11-Pad2) -> /REV_SW
- R12 pad 1: /Headlight_SW -> GND
- R12 pad 2: Net-(R12-Pad2) -> /FOR_SW
- R13 pad 1: GND -> Net-(J6-Pad2)
- R13 pad 2: /HZD_SW -> Net-(C8-Pad2)
- R14 pad 1: /CRUZ_ST -> Net-(J7-Pad2)
- R14 pad 2: GND -> /FOR_SW
- R15 pad 1: GND -> Net-(J8-Pad2)
- R15 pad 2: /CRUZ_EN -> /REV_SW
- R16 pad 1: GND -> GNDPWR
- R16 pad 2: /LEFT_SW -> /RIGHT_BLINK
- R17 pad 1: GND -> GNDPWR
- R17 pad 2: /RIGHT_SW -> /LEFT_BLINK
- R18 pad 1: +5V -> GNDPWR
- R18 pad 2: Net-(D0-Pad2) -> /RIGHT_BLINK
- R19 pad 1: GND -> GNDPWR
- R19 pad 2: /REV_SW -> /LEFT_BLINK
- R2 pad 1: Net-(D3-Pad1) -> /CRUZ_ST
- R20 pad 1: GND -> +12V
- R20 pad 2: /FOR_SW -> /HEADLIGHT_SW
- R21 pad 1: GND -> +12V
- R21 pad 2: /Headlight_SW -> Net-(J14-Pad1)
- R22 pad 1: +3V3 -> Net-(J9-Pad1)
- R22 pad 2: Net-(BL1-Pad7) -> +12V
- R23 pad 1: /BlinkTimer/TRIGTHRES -> Net-(J10-Pad1)
- R23 pad 2: Net-(BL1-Pad7) -> +12V
- R9 pad 1: GND -> /TRIGTHRES
- R9 pad 2: /REGEN_SW -> Net-(BL1-Pad7)
- SW1 pad 1: /HZD_SW -> +3V3
- SW1 pad 2: +3V3 -> /CRUZ_ST
- SW2 pad 1: /CRUZ_ST -> +3V3
- SW2 pad 2: +3V3 -> /CRUZ_EN
- SW3 pad 1: /CRUZ_EN -> /REV_SW
- SW3 pad 2: +3V3 -> Net-(C8-Pad2)
- SW4 pad 1: /FOR_SW -> /REGEN_SW
- SW5 pad 1: /Headlight_SW -> /LEFT_BLINK
- SW5 pad 2: +3V3 -> /LIGHTSCLK
- TP3 pad 1: +5V -> +3V3
- TP4 pad 1: GND -> /LEFT_BLINK
- TP5 pad 1: +3V3 -> +12V
Routing:
- net Net-(D2-Pad1): track 0.00 -> 15.5 mm, vias 0 -> 1
- added copper zone on B.Cu, net +12V
- added copper zone on B.Cu, net GND
- added copper zone on B.Cu, net GNDPWR
Other:
- board outline added: 45.7 x 122.9 mm
- board text added: "Breaklight External"
- board text added: "Cruise Enable Indicator"
- board text added: "Cruise Enable Switch"
- board text added: "Cruise Set Indicator"
- board text added: "Cruise Set Switch"
- board text added: "F/R Switch"
- board text added: "Forward Indicator"
- board text added: "Hazard Switch"
- board text added: "Headlight External"
- board text added: "Left Blink External"
- board text added: "Left Blink Internal"
- board text added: "Neutral Indicator"
- board text added: "Power"
- board text added: "Regen Indicator"
- board text added: "Regen Switch"
- board text added: "Reverse Indicator"
- board text added: "Right Blink External"
- board text added: "Right Blink Internal"
- board text added: "Turn Signal Switch"

Commit message: is square now
Parts:
- moved LOGO1 306.8 mm to (-40.4, 60.5)
- moved LOGO2 279.9 mm to (-22.1, 59.4)
- moved D2 207.9 mm to (51.8, 39.9), turned to 180 degrees
- moved C3 202.5 mm to (49.0, 68.7)
- moved R2 202.5 mm to (44.6, 68.7)
- moved C4 202.5 mm to (48.9, 79.9)
- moved R10 202.5 mm to (44.3, 91.6)
- moved R3 202.5 mm to (44.1, 79.9)
- moved R6 196.0 mm to (69.1, 89.4)
- moved FB3 196.0 mm to (69.0, 84.3)
- moved R4 196.0 mm to (68.8, 79.0)
- moved R5 196.0 mm to (68.9, 81.8)
- moved C8 196.0 mm to (69.0, 86.6)
- moved BL1 190.9 mm to (69.3, 30.7)
- moved D7 190.9 mm to (69.3, 43.4)
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Routing:
- net Net-(J8-Pad2): track 0.00 -> 24.2 mm
- net Net-(D2-Pad1): track 15.5 -> 0.00 mm, vias 1 -> 0
- net /LEFT_BLINK: track 0.07 -> 0.64 mm
- removed copper zone on B.Cu, net GND
Other:
- board size 45.7 x 122.9 mm -> 80.5 x 99.3 mm
- board text added: "Breaklight"
- board text added: "Headlight"
- board text removed: "Breaklight External"
- board text removed: "Headlight External"

Commit message: Component layout
Parts:
- L Blink: renamed from TP4
- R Blink: renamed from TP7
- moved LOGO1 184.8 mm to (143.4, 79.4)
- moved LOGO2 175.3 mm to (144.3, 114.6), turned to 0 degrees
- moved R10 121.7 mm to (160.5, 127.5), turned to 90 degrees
- moved D2 102.8 mm to (152.1, 62.5)
- moved C12 97.4 mm to (143.3, 129.0), turned to 90 degrees
- moved C6 94.9 mm to (140.3, 97.8)
- moved R8 94.8 mm to (145.8, 95.8), turned to 90 degrees
- moved D6 94.6 mm to (134.6, 89.4)
- moved BL1 94.1 mm to (140.2, 92.6)
- moved C5 93.6 mm to (140.2, 87.4)
- moved C9 93.0 mm to (134.6, 95.8)
- moved R9 90.7 mm to (145.8, 89.4), turned to 90 degrees
- moved R5 86.4 mm to (150.4, 52.8), turned to 90 degrees
- moved C1 82.8 mm to (129.0, 119.6)
- moved C8 78.8 mm to (144.3, 110.0), turned to -90 degrees
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- renumbered TP5 to +12V, TP3 to +3V, TP6 to +5V, TP2 to GND, TP1 to GNDPWR, TP8 to Headlights, TP9 to Lights
Routing:
- net Net-(J8-Pad2): track 24.2 -> 0.00 mm
- net /LEFT_BLINK: track 0.64 -> 0.07 mm
- added copper zone on B.Cu, net GND
Other:
- board size 80.5 x 99.3 mm -> 80.3 x 98.8 mm
