File: Inputs.kicad_sch (KiCad schematic)
At the start: 28 parts

Commit message: Added BOM
Parts:
- C10, C11, C3, C4, C7, C8: value 0.01uF -> .01uF
Changed lines of the file:
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@@
       (effects (font (size 1.27 1.27)) hide)
     )
-    (property "Datasheet" "~" (at 95.885 100.711 0)
+    (property "Datasheet" "https://www.mouser.com/ProductDetail/71-CRCW0805100RFKEAH" (at 95.885 100.711 0)
       (effects (font (size 1.27 1.27)) hide)
     )
@@
       (effects (font (size 1.27 1.27)) hide)
     )
-    (property "Datasheet" "~" (at 241.935 90.17 0)
+    (property "Datasheet" "https://www.mouser.com/ProductDetail/71-CRCW0805100RFKEAH" (at 241.935 90.17 0)
       (effects (font (size 1.27 1.27)) hide)
     )
@@
       (effects (font (size 1.27 1.27)) (justify left))
     )
-    (property "Value" "0.01uF" (at 229.87 88.9 0)
+    (property "Value" ".01uF" (at 229.87 88.9 0)
       (effects (font (size 1.27 1.27)) (justify left))
     )
@@
       (effects (font (size 1.27 1.27)) hide)
     )
-    (property "Datasheet" "~" (at 227.965 88.265 0)
+    (property "Datasheet" "https://www.mouser.com/ProductDetail/KEMET/C0805C103J5RACTU?qs=Onq5MIl0ZjiJ615hCkQQ7A%3D%3D" (at 227.965 88.265 0)
       (effects (font (size 1.27 1.27)) hide)
     )
@@
       (effects (font (size 1.27 1.27)) hide)
     )
-    (property "Datasheet" "~" (at 144.145 99.06 0)
+    (property "Datasheet" "https://www.mouser.com/ProductDetail/71-CRCW0805100RFKEAH" (at 144.145 99.06 0)
       (effects (font (size 1.27 1.27)) hide)
     )
@@
       (effects (font (size 1.27 1.27)) (justify left))
     )
-    (property "Value" "0.01uF" (at 127.635 92.075 0)
+    (property "Value" ".01uF" (at 127.635 92.075 0)
       (effects (font (size 1.27 1.27)) (justify left))
     )
@@
       (effects (font (size 1.27 1.27)) hide)
     )
-    (property "Datasheet" "~" (at 135.89 93.345 0)
+    (property "Datasheet" "https://www.mouser.com/ProductDetail/KEMET/C0805C103J5RACTU?qs=Onq5MIl0ZjiJ615hCkQQ7A%3D%3D" (at 135.89 93.345 0)
       (effects (font (size 1.27 1.27)) hide)
     )
@@
       (effects (font (size 1.27 1.27)) hide)
     )
-    (property "Datasheet" "~" (at 236.855 64.77 0)
+    (property "Datasheet" "https://www.mouser.com/ProductDetail/71-CRCW0805100RFKEAH" (at 236.855 64.77 0)
       (effects (font (size 1.27 1.27)) hide)
     )
@@
       (effects (font (size 1.27 1.27)) hide)
     )
-    (property "Datasheet" "~" (at 189.103 88.138 0)
+    (property "Datasheet" "https://www.mouser.com/ProductDetail/603-RT0603FRE0710KL" (at 189.103 88.138 0)
       (effects (font (size 1.27 1.27)) hide)
     )
@@
       (effects (font (size 1.27 1.27)) (justify left))
     )
-    (property "Value" "0.01uF" (at 78.74 98.171 0)
+    (property "Value" ".01uF" (at 78.74 98.171 0)
       (effects (font (size 1.27 1.27)) (justify left))
     )
@@
       (effects (font (size 1.27 1.27)) hide)
     )
-    (property "Datasheet" "~" (at 87.63 96.901 0)
+    (property "Datasheet" "https://www.mouser.com/ProductDetail/KEMET/C0805C103J5RACTU?qs=Onq5MIl0ZjiJ615hCkQQ7A%3D%3D" (at 87.63 96.901 0)
       (effects (font (size 1.27 1.27)) hide)
     )
@@
       (effects (font (size 1.27 1.27)) hide)
     )
-    (property "Datasheet" "~" (at 220.98 88.265 0)
+    (property "Datasheet" "https://www.mouser.com/ProductDetail/603-RT0603FRE0710KL" (at 220.98 88.265 0)
       (effects (font (size 1.27 1.27)) hide)
     )
@@
       (effects (font (size 1.27 1.27)) hide)
     )
-    (property "Datasheet" "~" (at 44.45 93.345 0)
+    (property "Datasheet" "https://www.mouser.com/ProductDetail/603-RT0603FRE0710KL" (at 44.45 93.345 0)
       (effects (font (size 1.27 1.27)) hide)
     )
@@
       (effects (font (size 1.27 1.27)) hide)
     )
-    (property "Datasheet" "~" (at 91.44 96.901 0)
+    (property "Datasheet" "https://www.mouser.com/ProductDetail/603-RT0603FRE0710KL" (at 91.44 96.901 0)
       (effects (font (size 1.27 1.27)) hide)
     )
@@
       (effects (font (size 1.27 1.27)) (justify left))
     )
-    (property "Value" "0.01uF" (at 31.75 93.98 0)
+    (property "Value" ".01uF" (at 31.75 93.98 0)
       (effects (font (size 1.27 1.27)) (justify left))
     )
@@
       (effects (font (size 1.27 1.27)) hide)
     )
-    (property "Datasheet" "~" (at 40.64 92.71 0)
+    (property "Datasheet" "https://www.mouser.com/ProductDetail/KEMET/C0805C103J5RACTU?qs=Onq5MIl0ZjiJ615hCkQQ7A%3D%3D" (at 40.64 92.71 0)
       (effects (font (size 1.27 1.27)) hide)
     )
@@
       (effects (font (size 1.27 1.27)) hide)
     )
-    (property "Datasheet" "~" (at 48.26 99.06 0)
+    (property "Datasheet" "https://www.mouser.com/ProductDetail/71-CRCW0805100RFKEAH" (at 48.26 99.06 0)
       (effects (font (size 1.27 1.27)) hide)
     )
@@
       (effects (font (size 1.27 1.27)) hide)
     )
-    (property "Datasheet" "~" (at 139.7 93.345 0)
+    (property "Datasheet" "https://www.mouser.com/ProductDetail/603-RT0603FRE0710KL" (at 139.7 93.345 0)
       (effects (font (size 1.27 1.27)) hide)
     )
@@
       (effects (font (size 1.27 1.27)) hide)
     )
-    (property "Datasheet" "~" (at 204.978 88.519 0)
+    (property "Datasheet" "https://www.mouser.com/ProductDetail/603-RT0603FRE0710KL" (at 204.978 88.519 0)
       (effects (font (size 1.27 1.27)) hide)
     )
@@
       (effects (font (size 1.27 1.27)) hide)
     )
-    (property "Datasheet" "~" (at 239.395 78.105 0)
+    (property "Datasheet" "https://www.mouser.com/ProductDetail/71-CRCW0805100RFKEAH" (at 239.395 78.105 0)
       (effects (font (size 1.27 1.27)) hide)
     )
@@
       (effects (font (size 1.27 1.27)) (justify left))
     )
-    (property "Value" "0.01uF" (at 197.358 89.408 0)
+    (property "Value" ".01uF" (at 197.358 89.408 0)
       (effects (font (size 1.27 1.27)) (justify left))
     )
@@
       (effects (font (size 1.27 1.27)) hide)
     )
-    (property "Datasheet" "~" (at 196.088 88.138 0)
+    (property "Datasheet" "https://www.mouser.com/ProductDetail/KEMET/C0805C103J5RACTU?qs=Onq5MIl0ZjiJ615hCkQQ7A%3D%3D" (at 196.088 88.138 0)
       (effects (font (size 1.27 1.27)) hide)
     )
@@
       (effects (font (size 1.27 1.27)) (justify left))
     )
-    (property "Value" "0.01uF" (at 213.36 89.408 0)
+    (property "Value" ".01uF" (at 213.36 89.408 0)
       (effects (font (size 1.27 1.27)) (justify left))
     )
@@
       (effects (font (size 1.27 1.27)) hide)
     )
-    (property "Datasheet" "~" (at 212.09 88.138 0)
-      (effects (font (size 1.27 1.27)) hide)
-    )
+    (property "Datasheet" "https://www.mouser.com/ProductDetail/KEMET/C0805C103J5RACTU?qs=Onq5MIl0ZjiJ615hCkQQ7A%3D%3D" (at 212.09 88.138 0)
+      (effects (font (size 1.27 1.27)) hide)
+    )
