File: hardware/Buck_Converter_sch.kicad_sch (KiCad schematic)
At the start: 13 parts, among them U5 TPS5405DR

Commit message: Add shared KiCad libraries and update .gitmodules
Parts:
- C5, C6, C7, C9: footprint Capacitor_SMD:C_0603_1608Metric_Pad1.08x0.95mm_HandSolder -> Capacitor_SMD:C_0603_1608Metric
- R6: footprint Resistor_SMD:R_0603_1608Metric_Pad0.98x0.95mm_HandSolder -> Resistor_SMD:R_0603_1608Metric
